Commit message: 初步完成手眼标定程序

File: kinova_description/urdf/j2s7s300_standalone.xacro (robot description, xacro)
@@ -30,5 +30,5 @@
     </collision>
   </link>
-  <!-- for gazebo
+  <!-- for gazebo -->
   <link name="world"/>
   <joint name="connect_root_and_world" type="fixed">
@@ -36,5 +36,5 @@
     <parent link="world" />
     <origin xyz="0 0 0" rpy="0 0 0" />
-  </joint>  -->
+  </joint>
   <property name="robot_root" value="root" />
   <xacro:j2s7s300  base_parent="${robot_root}"/>

Commit message: gazebo加载莫名出问题只能加载出机械臂，不知道为什么gazebo中的文件被修改了，本版本已重新修正

File: kinova_description/urdf/j2s7s300_standalone.xacro (robot description, xacro)
@@ -30,5 +30,5 @@
     </collision>
   </link>
-  <!-- for gazebo -->
+  <!-- for gazebo
   <link name="world"/>
   <joint name="connect_root_and_world" type="fixed">
@@ -36,5 +36,5 @@
     <parent link="world" />
     <origin xyz="0 0 0" rpy="0 0 0" />
-  </joint>
+  </joint>  -->
   <property name="robot_root" value="root" />
   <xacro:j2s7s300  base_parent="${robot_root}"/>
