Commit message: 抓取放置框变大，还没测变大后的抓取情况

File: table_fix/urdf/table_fix.urdf (robot description, URDF)
Before this commit: robot table_fix, 3 links, 2 joints
Joints:
- joint left_fixed: origin xyz=0.2398 -0.517 0.21594 rpy=-1.5708 0 0 -> xyz=0.245 -0.175 0 rpy=0 0 0
- joint right_fixed: origin xyz=-0.2502 -0.517 0.21594 rpy=-1.5708 0 0 -> xyz=-0.245 -0.175 0 rpy=0 0 0
